File: main_pcb/kicad_docs/power_supply.sch (KiCad schematic (older format))
At the start: 21 parts, among them J5 ac_htr_pcb, J7 high_voltage_pcb, J8 dc_htr_pcb

Commit message: tweak DC heater, pcb, regenerate build files
Parts:
- C15, C16: value 4700u 10v -> 10000u 10v; footprint Capacitor_THT:CP_Radial_D12.5mm_P5.00mm -> Capacitor_THT:CP_Radial_D16.0mm_P7.50mm
- R21: value ? -> 3R3 5W
Changed lines of the file:
@@
 P 6450 5950
 F 0 "C15" H 6565 5996 50  0000 L CNN
-F 1 "4700u 10v" H 6565 5905 50  0000 L CNN
-F 2 "Capacitor_THT:CP_Radial_D12.5mm_P5.00mm" H 6450 5950 50  0001 C CNN
+F 1 "10000u 10v" H 6565 5905 50  0000 L CNN
+F 2 "Capacitor_THT:CP_Radial_D16.0mm_P7.50mm" H 6450 5950 50  0001 C CNN
 F 3 "~" H 6450 5950 50  0001 C CNN
 	1    6450 5950
@@
 P 7050 5350
 F 0 "R21" V 6843 5350 50  0000 C CNN
-F 1 "?" V 6934 5350 50  0000 C CNN
+F 1 "3R3 5W" V 6934 5350 50  0000 C CNN
 F 2 "Resistor_THT:R_Axial_DIN0617_L17.0mm_D6.0mm_P30.48mm_Horizontal" V 6980 5350 50  0001 C CNN
 F 3 "~" H 7050 5350 50  0001 C CNN
@@
 P 7650 5950
 F 0 "C16" H 7765 5996 50  0000 L CNN
-F 1 "4700u 10v" H 7765 5905 50  0000 L CNN
-F 2 "Capacitor_THT:CP_Radial_D12.5mm_P5.00mm" H 7650 5950 50  0001 C CNN
+F 1 "10000u 10v" H 7765 5905 50  0000 L CNN
+F 2 "Capacitor_THT:CP_Radial_D16.0mm_P7.50mm" H 7650 5950 50  0001 C CNN
 F 3 "~" H 7650 5950 50  0001 C CNN
 	1    7650 5950
