File: pcb/kicad_6_docs/it_is_the_champion.kicad_pcb (KiCad board)
At the start: 2 copper layers, 226.1 x 101.6 mm, 71 parts, among them J1 pre_in_pcb, J10 ps_dc_htr_in_pcb, J2 ts_pcb, J3 gain_pcb, J4 pre_out_pcb, J5 pre_hv_dc_in_pcb, J6 pre_dc_htr_in_pcb, J7 ps_hv_dc_out_pcb, J8 ps_dc_htr_out_pcb, J9 ps_hv_ac_in_pcb

Commit message: fix capacitor name typo
Parts:
- C4: value 22n MIMA MKP4 -> 22n WIMA MKP4
Changed lines of the file:
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@@
       (effects (font (size 1 1) (thickness 0.15)))
     )
-    (fp_text value "22n MIMA MKP4" (at 5 3.25) (layer "F.Fab")
+    (fp_text value "22n WIMA MKP4" (at 5 3.25) (layer "F.Fab")
       (effects (font (size 1 1) (thickness 0.15)))
     )
@@
     (fp_line (start 2.54 16.51) (end 9.935923 9.314927) (layer "B.SilkS") (width 0.12))
     (fp_line (start -9.929645 9.321621) (end -2.54 16.51) (layer "B.SilkS") (width 0.12))
-    (fp_arc (start 9.929644 -9.32162) (mid 12.663473 -5.012672) (end 13.619487 0) (layer "B.SilkS") (width 0.12))
+    (fp_arc (start 9.929644 -9.32162) (mid 12.663473 -5.012673) (end 13.619487 0) (layer "B.SilkS") (width 0.12))
     (fp_arc (start -9.929644 9.32162) (mid -13.619473 0.019721) (end -9.956598 -9.292825) (layer "B.SilkS") (width 0.12))
     (fp_arc (start 2.54 16.51) (mid 0 17.562102) (end -2.54 16.51) (layer "B.SilkS") (width 0.12))
@@
     (fp_line (start -2.54 -16.51) (end -9.956598 -9.292825) (layer "B.SilkS") (width 0.12))
     (fp_line (start 2.54 -16.51) (end 9.929644 -9.32162) (layer "B.SilkS") (width 0.12))
-    (fp_arc (start 9.929644 -9.32162) (mid 12.663473 -5.012672) (end 13.619487 0) (layer "B.SilkS") (width 0.12))
+    (fp_arc (start 9.929644 -9.32162) (mid 12.663473 -5.012673) (end 13.619487 0) (layer "B.SilkS") (width 0.12))
     (fp_arc (start -9.929644 9.32162) (mid -13.619473 0.019721) (end -9.956598 -9.292825) (layer "B.SilkS") (width 0.12))
     (fp_arc (start 2.54 16.51) (mid 0 17.562102) (end -2.54 16.51) (layer "B.SilkS") (width 0.12))

Commit message: tweak some values
Parts:
- C12, C13, C14, C15: value 100u 350v -> 220u 350v
- R19, R20: value 50R 5W -> 100R 5W
- R21: value ??? 5W -> 13R 5W
Changed lines of the file:
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@@
       (effects (font (size 1 1) (thickness 0.15)))
     )
-    (fp_text value "50R 5W" (at 15.24 4.12 90) (layer "F.Fab")
+    (fp_text value "100R 5W" (at 15.24 4.12 90) (layer "F.Fab")
       (effects (font (size 1 1) (thickness 0.15)))
     )
@@
       (effects (font (size 1 1) (thickness 0.15)))
     )
-    (fp_text value "??? 5W" (at 15.24 4.12 90) (layer "F.Fab")
+    (fp_text value "13R 5W" (at 15.24 4.12 90) (layer "F.Fab")
       (effects (font (size 1 1) (thickness 0.15)))
     )
@@
       (effects (font (size 1 1) (thickness 0.15)))
     )
-    (fp_text value "100u 350v" (at 3.75 10.25) (layer "F.Fab")
+    (fp_text value "220u 350v" (at 3.75 10.25) (layer "F.Fab")
       (effects (font (size 1 1) (thickness 0.15)))
     )
@@
       (effects (font (size 1 1) (thickness 0.15)))
     )
-    (fp_text value "100u 350v" (at 3.75 10.25) (layer "F.Fab")
+    (fp_text value "220u 350v" (at 3.75 10.25) (layer "F.Fab")
       (effects (font (size 1 1) (thickness 0.15)))
     )
@@
       (effects (font (size 1 1) (thickness 0.15)))
     )
-    (fp_text value "100u 350v" (at 3.75 10.25) (layer "F.Fab")
+    (fp_text value "220u 350v" (at 3.75 10.25) (layer "F.Fab")
       (effects (font (size 1 1) (thickness 0.15)))
     )
@@
       (effects (font (size 1 1) (thickness 0.15)))
     )
-    (fp_text value "50R 5W" (at 15.24 4.12 90) (layer "F.Fab")
+    (fp_text value "100R 5W" (at 15.24 4.12 90) (layer "F.Fab")
       (effects (font (size 1 1) (thickness 0.15)))
     )
@@
       (effects (font (size 1 1) (thickness 0.15)))
     )
-    (fp_text value "100u 350v" (at 3.75 10.25) (layer "F.Fab")
-      (effects (font (size 1 1) (thickness 0.15)))
-    )
+    (fp_text value "220u 350v" (at 3.75 10.25) (layer "F.Fab")
+      (effects (font (size 1 1) (thickness 0.15)))
+    )
