File: pcb/kicad_6_docs/it_is_the_champion.kicad_sch (KiCad schematic)
At the start: 18 parts

Commit message: tweak some values
Parts:
- #F1: value 2A sb -> 1A sb
Other:
- note added: "120 VAC in"
- note added: "390mA @ idle 410mA @ max"
- note removed: "???mA @ idle ???mA @ max"
Changed lines of the file:
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@@
     (stroke (width 0) (type default) (color 0 0 0 0))
   )
-  (text "All voltages and \ncurrents approximate." (at 195.58 139.7 0)
+  (text "All voltages and \ncurrents approximate." (at 194.31 139.7 0)
     (effects (font (size 2.9972 2.9972)) (justify left bottom))
   )
@@
     (effects (font (size 2.9972 2.9972)) (justify left bottom))
   )
-  (text "???mA @ idle\n???mA @ max" (at 25.4 87.63 0)
+  (text "120 VAC in" (at 24.13 77.47 0)
+    (effects (font (size 2.9972 2.9972)) (justify left bottom))
+  )
+  (text "390mA @ idle\n410mA @ max" (at 25.4 86.36 0)
     (effects (font (size 2.0066 2.0066)) (justify left bottom))
   )
@@
     (in_bom yes) (on_board yes)
     (property "Reference" "#F1" (id 0) (at 55.88 97.8662 90))
-    (property "Value" "2A sb" (id 1) (at 55.88 100.1776 90))
+    (property "Value" "1A sb" (id 1) (at 55.88 100.1776 90))
     (property "Footprint" "" (id 2) (at 55.88 101.092 90)
       (effects (font (size 1.27 1.27)) hide)
@@
     )
     (path "/00000000-0000-0000-0000-00006115e9cb"
-      (reference "#F1") (unit 1) (value "2A sb") (footprint "")
+      (reference "#F1") (unit 1) (value "1A sb") (footprint "")
     )
     (path "/00000000-0000-0000-0000-00006111610f/00000000-0000-0000-0000-00006112f588"
@@
       (reference "#PWR0102") (unit 1) (value "Earth") (footprint "")
     )
-    (path "/00000000-0000-0000-0000-000061116f52/00000000-0000-0000-0000-000061f4e050"
-      (reference "#PWR0103") (unit 1) (value "Earth") (footprint "")
-    )
     (path "/00000000-0000-0000-0000-00006111610f/00000000-0000-0000-0000-000061b42153"
       (reference "#PWR0104") (unit 1) (value "GND3") (footprint "")
@@
     )
     (path "/00000000-0000-0000-0000-000061116994/00000000-0000-0000-0000-000061288f09"
-      (reference "#R3") (unit 1) (value "330R 25W") (footprint "Resistor_THT:R_Axial_Power_L48.0mm_W12.5mm_P60.96mm")
+      (reference "#R3") (unit 1) (value "390R 25W") (footprint "Resistor_THT:R_Axial_Power_L48.0mm_W12.5mm_P60.96mm")
     )
     (path "/00000000-0000-0000-0000-000061116994/00000000-0000-0000-0000-000061287cef"
-      (reference "#R4") (unit 1) (value "470R 5W") (footprint "Resistor_THT:R_Axial_DIN0414_L11.9mm_D4.5mm_P20.32mm_Horizontal")
+      (reference "#R4") (unit 1) (value "470R 2W") (footprint "Resistor_THT:R_Axial_DIN0414_L11.9mm_D4.5mm_P20.32mm_Horizontal")
     )
     (path "/00000000-0000-0000-0000-000061871bcb"
@@
       (reference "#T1") (unit 1) (value "antek_AS-1T175") (footprint "")
     )
-    (path "/00000000-0000-0000-0000-000061116f52/fb048223-89cc-497a-aa13-7584c82def6c"
-      (reference "#T2") (unit 1) (value "antek_AN-0115") (footprint "")
-    )
     (path "/00000000-0000-0000-0000-000061116994/da7f0dcc-a3b9-4032-812d-1070372a71d9"
       (reference "#T3") (unit 1) (value "edcor_GXSE15-8-5k") (footprint "")
@@
     )
     (path "/00000000-0000-0000-0000-000061116f52/00000000-0000-0000-0000-000061dbdae1"
-      (reference "C12") (unit 1) (value "100u 350v") (footprint "Capacitor_THT:CP_Radial_D18.0mm_P7.50mm")
+      (reference "C12") (unit 1) (value "220u 350v") (footprint "Capacitor_THT:CP_Radial_D18.0mm_P7.50mm")
     )
     (path "/00000000-0000-0000-0000-000061116f52/00000000-0000-0000-0000-000061dbe171"
-      (reference "C13") (unit 1) (value "100u 350v") (footprint "Capacitor_THT:CP_Radial_D18.0mm_P7.50mm")
+      (reference "C13") (unit 1) (value "220u 350v") (footprint "Capacitor_THT:CP_Radial_D18.0mm_P7.50mm")
     )
     (path "/00000000-0000-0000-0000-000061116f52/00000000-0000-0000-0000-000061de3470"
-      (reference "C14") (unit 1) (value "100u 350v") (footprint "Capacitor_THT:CP_Radial_D18.0mm_P7.50mm")
+      (reference "C14") (unit 1) (value "220u 350v") (footprint "Capacitor_THT:CP_Radial_D18.0mm_P7.50mm")
     )
     (path "/00000000-0000-0000-0000-000061116f52/00000000-0000-0000-0000-000061161cd6"
-      (reference "C15") (unit 1) (value "100u 350v") (footprint "Capacitor_THT:CP_Radial_D18.0mm_P7.50mm")
+      (reference "C15") (unit 1) (value "220u 350v") (footprint "Capacitor_THT:CP_Radial_D18.0mm_P7.50mm")
     )
     (path "/00000000-0000-0000-0000-000061116f52/00000000-0000-0000-0000-0000612fa2a2"
@@
     )
     (path "/00000000-0000-0000-0000-000061116f52/00000000-0000-0000-0000-00006129af6f"
-      (reference "R19") (unit 1) (value "50R 5W") (footprint "Resistor_THT:R_Axial_DIN0617_L17.0mm_D6.0mm_P30.48mm_Horizontal")
+      (reference "R19") (unit 1) (value "100R 5W") (footprint "Resistor_THT:R_Axial_DIN0617_L17.0mm_D6.0mm_P30.48mm_Horizontal")
     )
     (path "/00000000-0000-0000-0000-000061116f52/00000000-0000-0000-0000-000061de3a1f"
-      (reference "R20") (unit 1) (value "50R 5W") (footprint "Resistor_THT:R_Axial_DIN0617_L17.0mm_D6.0mm_P30.48mm_Horizontal")
+      (reference "R20") (unit 1) (value "100R 5W") (footprint "Resistor_THT:R_Axial_DIN0617_L17.0mm_D6.0mm_P30.48mm_Horizontal")
     )
     (path "/00000000-0000-0000-0000-000061116f52/00000000-0000-0000-0000-00006164163f"
-      (reference "R21") (unit 1) (value "??? 5W") (footprint "Resistor_THT:R_Axial_DIN0617_L17.0mm_D6.0mm_P30.48mm_Horizontal")
+      (reference "R21") (unit 1) (value "13R 5W") (footprint "Resistor_THT:R_Axial_DIN0617_L17.0mm_D6.0mm_P30.48mm_Horizontal")
     )
     (path "/00000000-0000-0000-0000-00006111610f/1c09aa33-b1b8-4383-bff4-8ce92d45169a"
