File: pcb/kicad_6_docs/power_amp.kicad_sch (KiCad schematic)
At the start: 8 parts

Commit message: tweak some values
Parts:
- #R3: value 330R 25W -> 390R 25W
- #R4: value 470R 5W -> 470R 2W
Connections:
- net GND2: no longer #MASTER1.1
- net speaker_out_+: now also #T3.white; no longer #T3.orange
- net speaker_out_-: now also #T3.orange; no longer #T3.white
- new net pa_signal_gnd: #MASTER1.1
Other:
- note added: "235VDC"
- note added: "470VDC"
- note added: "70mA"
- note removed: "240VDC"
- note removed: "480VDC"
- note removed: "80mA"
Changed lines of the file:
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@@
   (junction (at 93.98 104.14) (diameter 0) (color 0 0 0 0)
   )
-  (junction (at 83.82 114.3) (diameter 0) (color 0 0 0 0)
-  )
   (junction (at 121.92 114.3) (diameter 0) (color 0 0 0 0)
   )
   (junction (at 121.92 142.24) (diameter 0) (color 0 0 0 0)
   )
-  (junction (at 93.98 142.24) (diameter 0) (color 0 0 0 0)
-  )
   (junction (at 121.92 146.05) (diameter 0) (color 0 0 0 0)
   )
@@
   (junction (at 121.92 139.7) (diameter 0) (color 0 0 0 0)
   )
-  (no_connect (at 162.56 68.58))
+  (no_connect (at 142.24 66.04))
   (wire (pts (xy 121.92 142.24) (xy 93.98 142.24))
     (stroke (width 0) (type default) (color 0 0 0 0))
   )
-  (wire (pts (xy 124.46 60.96) (xy 124.46 91.44))
+  (wire (pts (xy 124.46 73.66) (xy 124.46 91.44))
     (stroke (width 0) (type default) (color 0 0 0 0))
   )
@@
     (stroke (width 0) (type default) (color 0 0 0 0))
   )
+  (wire (pts (xy 144.78 101.6) (xy 149.86 101.6))
+    (stroke (width 0) (type default) (color 0 0 0 0))
+  )
   (wire (pts (xy 134.62 107.95) (xy 132.08 107.95))
     (stroke (width 0) (type default) (color 0 0 0 0))
@@
     (stroke (width 0) (type default) (color 0 0 0 0))
   )
-  (wire (pts (xy 208.28 63.5) (xy 203.2 63.5))
+  (wire (pts (xy 187.96 60.96) (xy 182.88 60.96))
     (stroke (width 0) (type default) (color 0 0 0 0))
   )
@@
     (stroke (width 0) (type default) (color 0 0 0 0))
   )
-  (wire (pts (xy 83.82 114.3) (xy 83.82 142.24))
-    (stroke (width 0) (type default) (color 0 0 0 0))
-  )
-  (wire (pts (xy 93.98 142.24) (xy 83.82 142.24))
-    (stroke (width 0) (type default) (color 0 0 0 0))
-  )
   (wire (pts (xy 143.51 129.54) (xy 143.51 127))
     (stroke (width 0) (type default) (color 0 0 0 0))
@@
     (stroke (width 0) (type default) (color 0 0 0 0))
   )
-  (wire (pts (xy 162.56 60.96) (xy 124.46 60.96))
+  (wire (pts (xy 142.24 73.66) (xy 124.46 73.66))
     (stroke (width 0) (type default) (color 0 0 0 0))
   )
@@
     (stroke (width 0) (type default) (color 0 0 0 0))
   )
-  (wire (pts (xy 148.59 101.6) (xy 144.78 101.6))
-    (stroke (width 0) (type default) (color 0 0 0 0))
-  )
-  (wire (pts (xy 203.2 73.66) (xy 208.28 73.66))
-    (stroke (width 0) (type default) (color 0 0 0 0))
-  )
-  (wire (pts (xy 157.48 76.2) (xy 162.56 76.2))
+  (wire (pts (xy 182.88 71.12) (xy 187.96 71.12))
+    (stroke (width 0) (type default) (color 0 0 0 0))
+  )
+  (wire (pts (xy 139.7 58.42) (xy 142.24 58.42))
     (stroke (width 0) (type default) (color 0 0 0 0))
   )
@@
     (stroke (width 0) (type default) (color 0 0 0 0))
   )
-  (text "480VDC" (at 147.32 73.66 0)
+  (text "470VDC" (at 128.27 55.88 0)
     (effects (font (size 1.27 1.27)) (justify left bottom))
   )
-  (text "240VDC" (at 148.59 99.06 0)
+  (text "235VDC" (at 148.59 99.06 0)
     (effects (font (size 1.27 1.27)) (justify left bottom))
   )
-  (text "80mA" (at 113.03 133.35 0)
+  (text "70mA" (at 113.03 134.62 0)
     (effects (font (size 1.27 1.27)) (justify left bottom))
   )
@@
     (effects (font (size 2.9972 2.9972)) (justify left bottom))
   )
-  (hierarchical_label "pa_b+1_in" (shape input) (at 157.48 76.2 180)
+  (hierarchical_label "pa_b+1_in" (shape input) (at 139.7 58.42 180)
     (effects (font (size 1.27 1.27)) (justify right))
   )
@@
     (effects (font (size 1.27 1.27)) (justify left))
   )
-  (hierarchical_label "pa_b+2_in" (shape input) (at 148.59 101.6 0)
-    (effects (font (size 1.27 1.27)) (justify left))
-  )
-  (hierarchical_label "speaker_out_+" (shape output) (at 208.28 63.5 0)
-    (effects (font (size 1.27 1.27)) (justify left))
-  )
-  (hierarchical_label "speaker_out_-" (shape output) (at 208.28 73.66 0)
+  (hierarchical_label "pa_b+2_in" (shape input) (at 149.86 101.6 0)
+    (effects (font (size 1.27 1.27)) (justify left))
+  )
+  (hierarchical_label "speaker_out_+" (shape output) (at 187.96 60.96 0)
+    (effects (font (size 1.27 1.27)) (justify left))
+  )
+  (hierarchical_label "speaker_out_-" (shape output) (at 187.96 71.12 0)
     (effects (font (size 1.27 1.27)) (justify left))
   )
@@
     (in_bom yes) (on_board yes)
     (property "Reference" "#R4" (id 0) (at 140.97 96.3422 90))
-    (property "Value" "470R 5W" (id 1) (at 140.97 98.6536 90))
+    (property "Value" "470R 2W" (id 1) (at 140.97 98.6536 90))
     (property "Footprint" "Resistor_THT:R_Axial_DIN0414_L11.9mm_D4.5mm_P20.32mm_Horizontal" (id 2) (at 140.97 99.822 90)
       (effects (font (size 1.27 1.27)) hide)
@@
       (effects (font (size 1.27 1.27)) (justify left))
     )
-    (property "Value" "330R 25W" (id 1) (at 123.698 134.493 0)
+    (property "Value" "390R 25W" (id 1) (at 123.698 134.493 0)
       (effects (font (size 1.27 1.27)) (justify left))
     )
@@
     (pin "7")
   )
-  (symbol (lib_id "custom_symbols:edcor_GXSE15-x-yk") (at 184.15 66.04 0) (unit 1)
+  (symbol (lib_id "custom_symbols:edcor_GXSE15-x-yk") (at 163.83 68.58 0) (mirror x) (unit 1)
     (in_bom yes) (on_board yes) (fields_autoplaced)
-    (property "Reference" "#T3" (id 0) (at 182.88 53.34 0)
+    (property "Reference" "#T3" (id 0) (at 162.56 50.8 0)
       (effects (font (size 1.778 1.778)))
     )
-    (property "Value" "edcor_GXSE15-8-5k" (id 1) (at 182.88 57.15 0)
+    (property "Value" "edcor_GXSE15-8-5k" (id 1) (at 162.56 54.61 0)
       (effects (font (size 1.778 1.778)))
     )
-    (property "Footprint" "" (id 2) (at 182.88 66.04 0)
+    (property "Footprint" "" (id 2) (at 162.56 68.58 0)
       (effects (font (size 1.524 1.524)))
     )
-    (property "Datasheet" "" (id 3) (at 182.88 66.04 0)
+    (property "Datasheet" "" (id 3) (at 162.56 68.58 0)
       (effects (font (size 1.524 1.524)))
     )
