File: pcb/kicad_6_docs/power_supply.kicad_sch (KiCad schematic)
At the start: 28 parts, among them J10 ps_dc_htr_in_pcb, J7 ps_hv_dc_out_pcb, J8 ps_dc_htr_out_pcb, J9 ps_hv_ac_in_pcb

Commit message: tweak some values
Parts:
- removed #T2: antek_AN-0115, symbol custom_symbols:antek_AN-0115
- C12, C13, C14, C15: value 100u 350v -> 220u 350v
- R19, R20: value 50R 5W -> 100R 5W
- R21: value ??? 5W -> 13R 5W
Connections:
- net Earth: no longer #T1.blue_2, #T1.green_1
- net ps_ac_htr_out_1: now also #J10.2 (Pin_2)
- net ps_ac_htr_out_2: now also #J10.1 (Pin_1)
- new net: #T1.blue_2, #T1.green_1
Other:
- note added: "235VDC"
- note added: "470VDC"
- note added: "Heater windings may also be (blue, green) and (brown, orange) from the factory"
- note added: "R21 may need to be adjusted to get the DC heaters within 10% of 12.6V"
- note removed: "240VDC"
- note removed: "480VDC"
