File: pcb/kicad_6/it_is_the_champion.kicad_pcb (KiCad board)
At the start: 2 copper layers, 226.1 x 101.6 mm, 71 parts, among them J1 pre_in_pcb, J10 ps_dc_htr_in_pcb, J2 ts_pcb, J3 gain_pcb, J4 pre_out_pcb, J5 pre_hv_dc_in_pcb, J6 pre_dc_htr_in_pcb, J7 ps_hv_dc_out_pcb, J8 ps_dc_htr_out_pcb, J9 ps_hv_ac_in_pcb

Commit message: Tweaks to KiCad pcb project
Parts:
- moved H3 90.4 mm to (256.5, 141.0)
- moved H2 90.4 mm to (256.5, 49.5)
- moved J3 90.4 mm to (213.4, 61.5)
- moved C10 90.4 mm to (177.8, 130.8)
- moved C12 90.4 mm to (77.5, 97.5)
- moved C13 90.4 mm to (97.8, 97.5)
- moved C16 90.4 mm to (50.8, 96.3)
- moved C17 90.4 mm to (50.8, 78.5)
- moved C3 90.4 mm to (218.6, 74.9)
- moved C4 90.4 mm to (218.6, 67.3)
- moved C9 90.4 mm to (125.7, 75.1)
- moved D1 90.4 mm to (43.2, 111.8)
- moved D3 90.4 mm to (67.3, 111.1)
- moved D5 90.4 mm to (77.5, 111.1)
- moved D6 90.4 mm to (72.4, 134.6)
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