File: pcb/kicad_6/it_is_the_champion.kicad_sch (KiCad schematic)
At the start: 18 parts

Commit message: Tweaks to KiCad pcb project
Parts:
- #F1: value 1A sb -> 2A sb
- H1, H10, H11, H12, H2, H3, H4, H5, H6, H7, H8, H9: now left out of the parts list
Changed lines of the file:
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@@
   (title_block
     (title "It is the Champion")
-    (date "2021-12-30")
+    (date "2022-07-16")
     (rev "0.1")
     (comment 1 "creativecommons.org/licenses/by/4.0/")
@@
     (stroke (width 0) (type default) (color 0 0 0 0))
   )
+  (bus (pts (xy 146.05 67.31) (xy 146.05 100.33))
+    (stroke (width 0) (type default) (color 0 0 0 0))
+  )
   (wire (pts (xy 223.52 43.18) (xy 226.06 43.18))
     (stroke (width 0) (type default) (color 0 0 0 0))
@@
     (stroke (width 0) (type default) (color 0 0 0 0))
   )
-  (bus (pts (xy 165.1 54.61) (xy 165.1 57.15))
-    (stroke (width 0) (type default) (color 0 0 0 0))
-  )
   (wire (pts (xy 81.28 43.18) (xy 78.74 43.18))
     (stroke (width 0) (type default) (color 0 0 0 0))
@@
     (stroke (width 0) (type default) (color 0 0 0 0))
   )
+  (bus (pts (xy 146.05 62.23) (xy 146.05 64.77))
+    (stroke (width 0) (type default) (color 0 0 0 0))
+  )
   (wire (pts (xy 78.74 35.56) (xy 100.33 35.56))
     (stroke (width 0) (type default) (color 0 0 0 0))
@@
     (stroke (width 0) (type default) (color 0 0 0 0))
   )
-  (bus (pts (xy 146.05 107.95) (xy 146.05 110.49))
-    (stroke (width 0) (type default) (color 0 0 0 0))
-  )
   (wire (pts (xy 132.08 35.56) (xy 176.53 35.56))
     (stroke (width 0) (type default) (color 0 0 0 0))
@@
     (stroke (width 0) (type default) (color 0 0 0 0))
   )
-  (bus (pts (xy 146.05 67.31) (xy 146.05 100.33))
-    (stroke (width 0) (type default) (color 0 0 0 0))
-  )
   (wire (pts (xy 219.71 46.99) (xy 219.71 43.18))
     (stroke (width 0) (type default) (color 0 0 0 0))
@@
     (stroke (width 0) (type default) (color 0 0 0 0))
   )
-  (bus (pts (xy 146.05 55.88) (xy 146.05 59.69))
-    (stroke (width 0) (type default) (color 0 0 0 0))
-  )
   (wire (pts (xy 226.06 39.37) (xy 223.52 39.37))
     (stroke (width 0) (type default) (color 0 0 0 0))
@@
     (stroke (width 0) (type default) (color 0 0 0 0))
   )
-  (bus (pts (xy 146.05 62.23) (xy 146.05 64.77))
+  (bus (pts (xy 146.05 59.69) (xy 146.05 62.23))
     (stroke (width 0) (type default) (color 0 0 0 0))
   )
@@
     (stroke (width 0) (type default) (color 0 0 0 0))
   )
-  (bus (pts (xy 165.1 129.54) (xy 165.1 132.08))
-    (stroke (width 0) (type default) (color 0 0 0 0))
-  )
   (bus (pts (xy 146.05 102.87) (xy 146.05 105.41))
     (stroke (width 0) (type default) (color 0 0 0 0))
@@
   )
   (wire (pts (xy 83.82 43.18) (xy 100.33 43.18))
-    (stroke (width 0) (type default) (color 0 0 0 0))
-  )
-  (bus (pts (xy 146.05 59.69) (xy 146.05 62.23))
     (stroke (width 0) (type default) (color 0 0 0 0))
   )
@@
     (in_bom yes) (on_board yes)
     (property "Reference" "#F1" (id 0) (at 55.88 97.8662 90))
-    (property "Value" "1A sb" (id 1) (at 55.88 100.1776 90))
+    (property "Value" "2A sb" (id 1) (at 55.88 100.1776 90))
     (property "Footprint" "" (id 2) (at 55.88 101.092 90)
       (effects (font (size 1.27 1.27)) hide)
@@
   )
   (symbol (lib_id "Mechanical:MountingHole") (at 60.96 177.8 0) (unit 1)
-    (in_bom yes) (on_board yes)
+    (in_bom no) (on_board yes)
     (property "Reference" "H5" (id 0) (at 63.5 176.6316 0)
       (effects (font (size 1.27 1.27)) (justify left))
@@
   )
   (symbol (lib_id "Mechanical:MountingHole") (at 78.74 177.8 0) (unit 1)
-    (in_bom yes) (on_board yes)
+    (in_bom no) (on_board yes)
     (property "Reference" "H7" (id 0) (at 81.28 176.6316 0)
       (effects (font (size 1.27 1.27)) (justify left))
@@
   )
   (symbol (lib_id "Mechanical:MountingHole") (at 60.96 190.5 0) (unit 1)
-    (in_bom yes) (on_board yes)
+    (in_bom no) (on_board yes)
     (property "Reference" "H6" (id 0) (at 63.5 189.3316 0)
       (effects (font (size 1.27 1.27)) (justify left))
@@
   )
   (symbol (lib_id "Mechanical:MountingHole") (at 78.74 190.5 0) (unit 1)
-    (in_bom yes) (on_board yes)
+    (in_bom no) (on_board yes)
     (property "Reference" "H8" (id 0) (at 81.28 189.3316 0)
       (effects (font (size 1.27 1.27)) (justify left))
@@
   )
   (symbol (lib_id "Mechanical:MountingHole") (at 96.52 177.8 0) (unit 1)
-    (in_bom yes) (on_board yes)
+    (in_bom no) (on_board yes)
     (property "Reference" "H9" (id 0) (at 99.06 176.6316 0)
       (effects (font (size 1.27 1.27)) (justify left))
@@
   )
   (symbol (lib_id "Mechanical:MountingHole") (at 114.3 177.8 0) (unit 1)
-    (in_bom yes) (on_board yes)
+    (in_bom no) (on_board yes)
     (property "Reference" "H11" (id 0) (at 116.84 176.6316 0)
       (effects (font (size 1.27 1.27)) (justify left))
@@
   )
   (symbol (lib_id "Mechanical:MountingHole") (at 96.52 190.5 0) (unit 1)
-    (in_bom yes) (on_board yes)
+    (in_bom no) (on_board yes)
     (property "Reference" "H10" (id 0) (at 99.06 189.3316 0)
       (effects (font (size 1.27 1.27)) (justify left))
@@
   )
   (symbol (lib_id "Mechanical:MountingHole") (at 114.3 190.5 0) (unit 1)
-    (in_bom yes) (on_board yes)
+    (in_bom no) (on_board yes)
     (property "Reference" "H12" (id 0) (at 116.84 189.3316 0)
       (effects (font (size 1.27 1.27)) (justify left))
@@
   )
   (symbol (lib_id "Mechanical:MountingHole") (at 25.4 177.8 0) (unit 1)
-    (in_bom yes) (on_board yes)
+    (in_bom no) (on_board yes)
     (property "Reference" "H1" (id 0) (at 27.94 176.6316 0)
       (effects (font (size 1.27 1.27)) (justify left))
@@
   )
   (symbol (lib_id "Mechanical:MountingHole") (at 43.18 177.8 0) (unit 1)
-    (in_bom yes) (on_board yes)
+    (in_bom no) (on_board yes)
     (property "Reference" "H3" (id 0) (at 45.72 176.6316 0)
       (effects (font (size 1.27 1.27)) (justify left))
@@
   )
   (symbol (lib_id "Mechanical:MountingHole") (at 25.4 190.5 0) (unit 1)
-    (in_bom yes) (on_board yes)
+    (in_bom no) (on_board yes)
     (property "Reference" "H2" (id 0) (at 27.94 189.3316 0)
       (effects (font (size 1.27 1.27)) (justify left))
@@
   )
   (symbol (lib_id "Mechanical:MountingHole") (at 43.18 190.5 0) (unit 1)
-    (in_bom yes) (on_board yes)
+    (in_bom no) (on_board yes)
     (property "Reference" "H4" (id 0) (at 45.72 189.3316 0)
       (effects (font (size 1.27 1.27)) (justify left))
@@
     )
     (path "/00000000-0000-0000-0000-00006115e9cb"
-      (reference "#F1") (unit 1) (value "1A sb") (footprint "")
+      (reference "#F1") (unit 1) (value "2A sb") (footprint "")
     )
     (path "/00000000-0000-0000-0000-00006111610f/00000000-0000-0000-0000-00006112f588"
