File: pcb/kicad_6/power_supply.kicad_sch (KiCad schematic)
At the start: 27 parts, among them J10 ps_dc_htr_in_pcb, J7 ps_hv_dc_out_pcb, J8 ps_dc_htr_out_pcb, J9 ps_hv_ac_in_pcb

Commit message: Tweaks to KiCad pcb project
Parts:
- J10, J7, J8, J9: now left out of the parts list
Changed lines of the file:
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@@
   (title_block
     (title "It is the Champion")
-    (date "2021-12-30")
+    (date "2022-07-16")
     (rev "0.1")
     (comment 1 "creativecommons.org/licenses/by/4.0/")
@@
   )
   (symbol (lib_id "Connector_Generic:Conn_01x02") (at 62.23 137.16 0) (mirror y) (unit 1)
-    (in_bom yes) (on_board yes)
+    (in_bom no) (on_board yes)
     (property "Reference" "J10" (id 0) (at 67.31 130.81 0)
       (effects (font (size 1.27 1.27)) (justify left))
@@
   )
   (symbol (lib_id "Connector_Generic:Conn_01x04") (at 120.65 43.18 0) (mirror y) (unit 1)
-    (in_bom yes) (on_board yes)
+    (in_bom no) (on_board yes)
     (property "Reference" "J9" (id 0) (at 125.73 34.29 0)
       (effects (font (size 1.27 1.27)) (justify left))
@@
   )
   (symbol (lib_id "Connector_Generic:Conn_01x02") (at 157.48 152.4 0) (unit 1)
-    (in_bom yes) (on_board yes)
+    (in_bom no) (on_board yes)
     (property "Reference" "J8" (id 0) (at 148.59 146.05 0)
       (effects (font (size 1.27 1.27)) (justify left))
@@
   )
   (symbol (lib_id "Connector_Generic:Conn_01x05") (at 229.87 53.34 0) (unit 1)
-    (in_bom yes) (on_board yes)
+    (in_bom no) (on_board yes)
     (property "Reference" "J7" (id 0) (at 223.52 41.91 0)
       (effects (font (size 1.27 1.27)) (justify left))
