File: pcb/kicad_6/preamp.kicad_sch (KiCad schematic)
At the start: 47 parts, among them J1 pre_in_pcb, J2 ts_pcb, J3 gain_pcb, J4 pre_out_pcb, J5 pre_hv_dc_in_pcb, J6 pre_dc_htr_in_pcb

Commit message: Tweaks to KiCad pcb project
Parts:
- J1, J2, J3, J4, J5, J6: now left out of the parts list
Changed lines of the file:
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@@
   (title_block
     (title "It is the Champion")
-    (date "2021-12-30")
+    (date "2022-07-16")
     (rev "0.1")
     (comment 1 "creativecommons.org/licenses/by/4.0/")
@@
   )
   (symbol (lib_id "Connector_Generic:Conn_01x02") (at 176.53 99.06 0) (mirror y) (unit 1)
-    (in_bom yes) (on_board yes)
+    (in_bom no) (on_board yes)
     (property "Reference" "J3" (id 0) (at 180.34 92.71 0)
       (effects (font (size 1.27 1.27)) (justify left))
@@
   )
   (symbol (lib_id "Connector_Generic:Conn_01x02") (at 198.12 194.31 0) (unit 1)
-    (in_bom yes) (on_board yes)
+    (in_bom no) (on_board yes)
     (property "Reference" "J6" (id 0) (at 193.04 187.96 0)
       (effects (font (size 1.27 1.27)) (justify left))
@@
   )
   (symbol (lib_id "Connector_Generic:Conn_01x02") (at 41.91 99.06 0) (mirror y) (unit 1)
-    (in_bom yes) (on_board yes)
+    (in_bom no) (on_board yes)
     (property "Reference" "J1" (id 0) (at 44.45 92.71 0)
       (effects (font (size 1.27 1.27)) (justify left))
@@
   )
   (symbol (lib_id "Connector_Generic:Conn_01x02") (at 304.8 82.55 0) (unit 1)
-    (in_bom yes) (on_board yes)
+    (in_bom no) (on_board yes)
     (property "Reference" "J4" (id 0) (at 300.99 76.2 0)
       (effects (font (size 1.27 1.27)) (justify left))
@@
   )
   (symbol (lib_id "Connector_Generic:Conn_01x03") (at 118.11 91.44 0) (unit 1)
-    (in_bom yes) (on_board yes)
+    (in_bom no) (on_board yes)
     (property "Reference" "J2" (id 0) (at 114.3 82.55 0)
       (effects (font (size 1.27 1.27)) (justify left))
@@
   )
   (symbol (lib_id "Connector_Generic:Conn_01x02") (at 318.77 39.37 0) (unit 1)
-    (in_bom yes) (on_board yes)
+    (in_bom no) (on_board yes)
     (property "Reference" "J5" (id 0) (at 313.69 33.02 0)
       (effects (font (size 1.27 1.27)) (justify left))
@@
     (pin "7")
     (pin "8")
+    (pin "1")
+    (pin "2")
+    (pin "3")
+    (pin "4")
+    (pin "5")
+    (pin "9")
   )
   (symbol (lib_id "custom_symbols:12AX7") (at 196.85 99.06 0) (unit 2)
@@
       (effects (font (size 1.27 1.27)) hide)
     )
+    (pin "6")
+    (pin "7")
+    (pin "8")
     (pin "1")
     (pin "2")
     (pin "3")
-  )
-  (symbol (lib_id "custom_symbols:12AX7") (at 148.59 177.8 0) (unit 3)
-    (in_bom yes) (on_board yes)
-    (property "Reference" "V1" (id 0) (at 152.4 167.64 0)
-      (effects (font (size 1.27 1.27)) (justify left))
-    )
-    (property "Value" "12AX7" (id 1) (at 152.4 170.18 0)
-      (effects (font (size 1.27 1.27)) (justify left))
-    )
-    (property "Footprint" "custom_footprints:belton_VT9-PT-C" (id 2) (at 155.448 187.96 0)
-      (effects (font (size 1.27 1.27)) hide)
-    )
-    (property "Datasheet" "" (id 3) (at 148.59 177.8 0)
-      (effects (font (size 1.27 1.27)) hide)
-    )
     (pin "4")
     (pin "5")
     (pin "9")
   )
+  (symbol (lib_id "custom_symbols:12AX7") (at 148.59 177.8 0) (unit 3)
+    (in_bom yes) (on_board yes)
+    (property "Reference" "V1" (id 0) (at 152.4 167.64 0)
+      (effects (font (size 1.27 1.27)) (justify left))
+    )
+    (property "Value" "12AX7" (id 1) (at 152.4 170.18 0)
+      (effects (font (size 1.27 1.27)) (justify left))
+    )
+    (property "Footprint" "custom_footprints:belton_VT9-PT-C" (id 2) (at 155.448 187.96 0)
+      (effects (font (size 1.27 1.27)) hide)
+    )
+    (property "Datasheet" "" (id 3) (at 148.59 177.8 0)
+      (effects (font (size 1.27 1.27)) hide)
+    )
+    (pin "6")
+    (pin "7")
+    (pin "8")
+    (pin "1")
+    (pin "2")
+    (pin "3")
+    (pin "4")
+    (pin "5")
+    (pin "9")
+  )
   (symbol (lib_id "custom_symbols:12AX7") (at 275.59 99.06 0) (unit 2)
     (in_bom yes) (on_board yes) (fields_autoplaced)
@@
       (effects (font (size 1.27 1.27)) hide)
     )
+    (pin "6")
+    (pin "7")
+    (pin "8")
     (pin "1")
     (pin "2")
     (pin "3")
+    (pin "4")
+    (pin "5")
+    (pin "9")
   )
   (symbol (lib_id "custom_symbols:12AX7") (at 237.49 99.06 0) (unit 1)
@@
     (pin "7")
     (pin "8")
-  )
-  (symbol (lib_id "custom_symbols:12AX7") (at 165.1 177.8 0) (unit 3)
-    (in_bom yes) (on_board yes)
-    (property "Reference" "V2" (id 0) (at 170.18 167.64 0)
-      (effects (font (size 1.27 1.27)) (justify left))
-    )
-    (property "Value" "12AX7" (id 1) (at 170.18 170.18 0)
-      (effects (font (size 1.27 1.27)) (justify left))
-    )
-    (property "Footprint" "custom_footprints:belton_VT9-PT-C" (id 2) (at 171.958 187.96 0)
-      (effects (font (size 1.27 1.27)) hide)
-    )
-    (property "Datasheet" "" (id 3) (at 165.1 177.8 0)
-      (effects (font (size 1.27 1.27)) hide)
-    )
+    (pin "1")
+    (pin "2")
+    (pin "3")
     (pin "4")
     (pin "5")
+    (pin "9")
+  )
+  (symbol (lib_id "custom_symbols:12AX7") (at 165.1 177.8 0) (unit 3)
+    (in_bom yes) (on_board yes)
+    (property "Reference" "V2" (id 0) (at 170.18 167.64 0)
+      (effects (font (size 1.27 1.27)) (justify left))
+    )
+    (property "Value" "12AX7" (id 1) (at 170.18 170.18 0)
+      (effects (font (size 1.27 1.27)) (justify left))
+    )
+    (property "Footprint" "custom_footprints:belton_VT9-PT-C" (id 2) (at 171.958 187.96 0)
+      (effects (font (size 1.27 1.27)) hide)
+    )
+    (property "Datasheet" "" (id 3) (at 165.1 177.8 0)
+      (effects (font (size 1.27 1.27)) hide)
+    )
+    (pin "6")
+    (pin "7")
+    (pin "8")
+    (pin "1")
+    (pin "2")
+    (pin "3")
+    (pin "4")
+    (pin "5")
